File: RPi_EthShield.sch (KiCad schematic (older format))
At the start: 18 parts, among them IC1 DS1233AZ-10+, J1 HR911105A, J2 RPi_GPIO, U1 ENC28J60x-SO, U2 LM1117-3.3, Y1 25MHz

Commit message: footprint for DS1233a fixed
Parts:
- IC1: footprint symbols:SOT230P700X180-4N -> EthShield:DS1233_SOT223
- J2: symbol Connector-ML:RPi_GPIO -> RPi_EthShield-rescue:RPi_GPIO-Connector-ML
Changed lines of the file:
@@
 $EndDescr
 $Comp
-L Connector-ML:RPi_GPIO J2
+L RPi_EthShield-rescue:RPi_GPIO-Connector-ML J2
 U 1 1 5516AE26
 P 7500 2700
@@
 F 0 "IC1" H 3450 3035 50  0000 C CNN
 F 1 "DS1233AZ-10+" H 3450 3126 50  0000 C CNN
-F 2 "symbols:SOT230P700X180-4N" H 4050 3600 50  0001 L CNN
+F 2 "EthShield:DS1233_SOT223" H 4050 3600 50  0001 L CNN
 F 3 "http://docs-emea.rs-online.com/webdocs/0f62/0900766b80f62e31.pdf" H 4050 3500 50  0001 L CNN
 F 4 "3.3V EconoReset" H 4050 3400 50  0001 L CNN "Description"
